File: Hardware/AFE Test design PCB/ADS1298_setup.sch (KiCad schematic (older format))
At the start: 17 parts

Commit message: update
Parts:
- gave numbers to parts that had none: 17
Changed lines of the file:
@@
 AR Path="/5D249131/5F07B13D" Ref="C?"  Part="1"
 AR Path="/5F07B13D" Ref="C?"  Part="1"
-AR Path="/5F050CC1/5F07B13D" Ref="C?"  Part="1"
-F 0 "C?" H 5040 6921 50  0000 L CNN
+AR Path="/5F050CC1/5F07B13D" Ref="C84"  Part="1"
+F 0 "C84" H 5040 6921 50  0000 L CNN
 F 1 "1nF" H 5040 6830 50  0000 L CNN
 F 2 "Capacitor_SMD:C_0805_2012Metric_Pad1.15x1.40mm_HandSolder" H 4963 6725 50  0001 C CNN
@@
 AR Path="/5D249131/5F07B144" Ref="C?"  Part="1"
 AR Path="/5F07B144" Ref="C?"  Part="1"
-AR Path="/5F050CC1/5F07B144" Ref="C?"  Part="1"
-F 0 "C?" H 2640 6921 50  0000 L CNN
+AR Path="/5F050CC1/5F07B144" Ref="C77"  Part="1"
+F 0 "C77" H 2640 6921 50  0000 L CNN
 F 1 "1uF" H 2640 6830 50  0000 L CNN
 F 2 "Capacitor_SMD:C_0805_2012Metric_Pad1.15x1.40mm_HandSolder" H 2563 6725 50  0001 C CNN
@@
 AR Path="/5D249131/5F07B14B" Ref="C?"  Part="1"
 AR Path="/5F07B14B" Ref="C?"  Part="1"
-AR Path="/5F050CC1/5F07B14B" Ref="C?"  Part="1"
-F 0 "C?" H 2990 6921 50  0000 L CNN
+AR Path="/5F050CC1/5F07B14B" Ref="C78"  Part="1"
+F 0 "C78" H 2990 6921 50  0000 L CNN
 F 1 "1uF" H 2990 6830 50  0000 L CNN
 F 2 "Capacitor_SMD:C_0805_2012Metric_Pad1.15x1.40mm_HandSolder" H 2913 6725 50  0001 C CNN
@@
 AR Path="/5D249131/5F07B152" Ref="C?"  Part="1"
 AR Path="/5F07B152" Ref="C?"  Part="1"
-AR Path="/5F050CC1/5F07B152" Ref="C?"  Part="1"
-F 0 "C?" H 3740 6921 50  0000 L CNN
+AR Path="/5F050CC1/5F07B152" Ref="C80"  Part="1"
+F 0 "C80" H 3740 6921 50  0000 L CNN
 F 1 "1uF" H 3740 6830 50  0000 L CNN
 F 2 "Capacitor_SMD:C_0805_2012Metric_Pad1.15x1.40mm_HandSolder" H 3663 6725 50  0001 C CNN
@@
 AR Path="/5D249131/5F07B159" Ref="C?"  Part="1"
 AR Path="/5F07B159" Ref="C?"  Part="1"
-AR Path="/5F050CC1/5F07B159" Ref="C?"  Part="1"
-F 0 "C?" H 4090 6921 50  0000 L CNN
+AR Path="/5F050CC1/5F07B159" Ref="C81"  Part="1"
+F 0 "C81" H 4090 6921 50  0000 L CNN
 F 1 "22uF" H 4090 6830 50  0000 L CNN
 F 2 "Capacitor_SMD:C_0805_2012Metric_Pad1.15x1.40mm_HandSolder" H 4013 6725 50  0001 C CNN
@@
 AR Path="/5D249131/5F07B172" Ref="C?"  Part="1"
 AR Path="/5F07B172" Ref="C?"  Part="1"
-AR Path="/5F050CC1/5F07B172" Ref="C?"  Part="1"
-F 0 "C?" H 4965 1696 50  0000 L CNN
+AR Path="/5F050CC1/5F07B172" Ref="C83"  Part="1"
+F 0 "C83" H 4965 1696 50  0000 L CNN
 F 1 "0.1u" H 4965 1605 50  0000 L CNN
 F 2 "Capacitor_SMD:C_0805_2012Metric_Pad1.15x1.40mm_HandSolder" H 4888 1500 50  0001 C CNN
@@
 AR Path="/5D249131/5F07B17D" Ref="C?"  Part="1"
 AR Path="/5F07B17D" Ref="C?"  Part="1"
-AR Path="/5F050CC1/5F07B17D" Ref="C?"  Part="1"
-F 0 "C?" H 3365 6921 50  0000 L CNN
+AR Path="/5F050CC1/5F07B17D" Ref="C79"  Part="1"
+F 0 "C79" H 3365 6921 50  0000 L CNN
 F 1 ".1uF" H 3365 6830 50  0000 L CNN
 F 2 "Capacitor_SMD:C_0805_2012Metric_Pad1.15x1.40mm_HandSolder" H 3288 6725 50  0001 C CNN
@@
 AR Path="/5D249131/5F07B1AE" Ref="C?"  Part="1"
 AR Path="/5F07B1AE" Ref="C?"  Part="1"
-AR Path="/5F050CC1/5F07B1AE" Ref="C?"  Part="1"
-F 0 "C?" H 5640 6921 50  0000 L CNN
+AR Path="/5F050CC1/5F07B1AE" Ref="C85"  Part="1"
+F 0 "C85" H 5640 6921 50  0000 L CNN
 F 1 "0.1uF" H 5640 6830 50  0000 L CNN
 F 2 "Capacitor_SMD:C_0805_2012Metric_Pad1.15x1.40mm_HandSolder" H 5563 6725 50  0001 C CNN
@@
 AR Path="/5D249131/5F07B1B5" Ref="C?"  Part="1"
 AR Path="/5F07B1B5" Ref="C?"  Part="1"
-AR Path="/5F050CC1/5F07B1B5" Ref="C?"  Part="1"
-F 0 "C?" H 6065 6921 50  0000 L CNN
+AR Path="/5F050CC1/5F07B1B5" Ref="C86"  Part="1"
+F 0 "C86" H 6065 6921 50  0000 L CNN
 F 1 "1uF" H 6065 6830 50  0000 L CNN
 F 2 "Capacitor_SMD:C_0805_2012Metric_Pad1.15x1.40mm_HandSolder" H 5988 6725 50  0001 C CNN
@@
 AR Path="/5D249131/5F07B1C2" Ref="#PWR?"  Part="1"
 AR Path="/5F07B1C2" Ref="#PWR?"  Part="1"
-AR Path="/5F050CC1/5F07B1C2" Ref="#PWR?"  Part="1"
-F 0 "#PWR?" H 5950 7125 50  0001 C CNN
+AR Path="/5F050CC1/5F07B1C2" Ref="#PWR070"  Part="1"
+F 0 "#PWR070" H 5950 7125 50  0001 C CNN
 F 1 "GND" H 5955 7202 50  0000 C CNN
 F 2 "" H 5950 7375 50  0001 C CNN
@@
 AR Path="/5D249131/5F07B1D6" Ref="#PWR?"  Part="1"
 AR Path="/5F07B1D6" Ref="#PWR?"  Part="1"
-AR Path="/5F050CC1/5F07B1D6" Ref="#PWR?"  Part="1"
-F 0 "#PWR?" H 1200 7200 50  0001 C CNN
+AR Path="/5F050CC1/5F07B1D6" Ref="#PWR066"  Part="1"
+F 0 "#PWR066" H 1200 7200 50  0001 C CNN
 F 1 "GND" H 1205 7277 50  0000 C CNN
 F 2 "" H 1200 7450 50  0001 C CNN
@@
 P 3450 3825
 AR Path="/5F07B21B" Ref="IC?"  Part="1"
-AR Path="/5F050CC1/5F07B21B" Ref="IC?"  Part="1"
-F 0 "IC?" H 3450 3900 50  0000 C CNN
+AR Path="/5F050CC1/5F07B21B" Ref="IC1"  Part="1"
+F 0 "IC1" H 3450 3900 50  0000 C CNN
 F 1 "ADS1298_By_Oliver" H 3450 3800 50  0000 C CNN
 F 2 "Package_QFP:TQFP-64_10x10mm_P0.5mm" H 3150 4275 50  0001 L BNN
@@
 AR Path="/5D249131/5F07B2D1" Ref="#PWR?"  Part="1"
 AR Path="/5F07B2D1" Ref="#PWR?"  Part="1"
-AR Path="/5F050CC1/5F07B2D1" Ref="#PWR?"  Part="1"
-F 0 "#PWR?" H 2450 5075 50  0001 C CNN
+AR Path="/5F050CC1/5F07B2D1" Ref="#PWR069"  Part="1"
+F 0 "#PWR069" H 2450 5075 50  0001 C CNN
 F 1 "GND" H 2455 5152 50  0000 C CNN
 F 2 "" H 2450 5325 50  0001 C CNN
@@
 AR Path="/5D249131/5F07B31F" Ref="#PWR?"  Part="1"
 AR Path="/5F07B31F" Ref="#PWR?"  Part="1"
-AR Path="/5F050CC1/5F07B31F" Ref="#PWR?"  Part="1"
-F 0 "#PWR?" H 2025 7200 50  0001 C CNN
+AR Path="/5F050CC1/5F07B31F" Ref="#PWR068"  Part="1"
+F 0 "#PWR068" H 2025 7200 50  0001 C CNN
 F 1 "GND" H 2030 7277 50  0000 C CNN
 F 2 "" H 2025 7450 50  0001 C CNN
@@
 AR Path="/5D249131/5F07B32D" Ref="#PWR?"  Part="1"
 AR Path="/5F07B32D" Ref="#PWR?"  Part="1"
-AR Path="/5F050CC1/5F07B32D" Ref="#PWR?"  Part="1"
-F 0 "#PWR?" H 6525 4525 50  0001 C CNN
+AR Path="/5F050CC1/5F07B32D" Ref="#PWR071"  Part="1"
+F 0 "#PWR071" H 6525 4525 50  0001 C CNN
 F 1 "GND" H 6530 4602 50  0000 C CNN
 F 2 "" H 6525 4775 50  0001 C CNN
@@
 AR Path="/5D249131/5F07B335" Ref="TP?"  Part="1"
 AR Path="/5F07B335" Ref="TP?"  Part="1"
-AR Path="/5F050CC1/5F07B335" Ref="TP?"  Part="1"
-F 0 "TP?" H 4150 1450 50  0000 L CNN
+AR Path="/5F050CC1/5F07B335" Ref="TP27"  Part="1"
+F 0 "TP27" H 4150 1450 50  0000 L CNN
 F 1 "TestPoint" H 4100 1350 50  0000 L CNN
 F 2 "TestPoint:TestPoint_Pad_D1.0mm" H 4300 1300 50  0001 C CNN
@@
 	1325 2825 2050 2825
 $Comp
-L Jumper:Jumper_3_Open JP?
+L Jumper:Jumper_3_Open JP35
 U 1 1 5D8D2D9A
 P 6525 4425
-F 0 "JP?" V 6479 4512 50  0000 L CNN
+F 0 "JP35" V 6479 4512 50  0000 L CNN
 F 1 "Jumper_3_Open" V 6570 4512 50  0000 L CNN
 F 2 "Jumper:SolderJumper-3_P1.3mm_Open_RoundedPad1.0x1.5mm" H 6525 4425 50  0001 C CNN
@@
 AR Path="/5D249131/5EFC0C47" Ref="#PWR?"  Part="1"
 AR Path="/5EFC0C47" Ref="#PWR?"  Part="1"
-AR Path="/5F050CC1/5EFC0C47" Ref="#PWR?"  Part="1"
-F 0 "#PWR?" H 6625 7125 50  0001 C CNN
+AR Path="/5F050CC1/5EFC0C47" Ref="#PWR072"  Part="1"
+F 0 "#PWR072" H 6625 7125 50  0001 C CNN
 F 1 "GND" H 6630 7202 50  0000 C CNN
 F 2 "" H 6625 7375 50  0001 C CNN
@@
 AR Path="/5D249131/5D96E834" Ref="C?"  Part="1"
 AR Path="/5D96E834" Ref="C?"  Part="1"
-AR Path="/5F050CC1/5D96E834" Ref="C?"  Part="1"
-F 0 "C?" H 2140 6946 50  0000 L CNN
+AR Path="/5F050CC1/5D96E834" Ref="C76"  Part="1"
+F 0 "C76" H 2140 6946 50  0000 L CNN
 F 1 "1uF" H 2140 6855 50  0000 L CNN
 F 2 "Capacitor_SMD:C_0805_2012Metric_Pad1.15x1.40mm_HandSolder" H 2063 6750 50  0001 C CNN
@@
 AR Path="/5D249131/5D96E8C2" Ref="C?"  Part="1"
 AR Path="/5D96E8C2" Ref="C?"  Part="1"
-AR Path="/5F050CC1/5D96E8C2" Ref="C?"  Part="1"
-F 0 "C?" H 1715 6946 50  0000 L CNN
+AR Path="/5F050CC1/5D96E8C2" Ref="C75"  Part="1"
+F 0 "C75" H 1715 6946 50  0000 L CNN
 F 1 "10uF" H 1715 6855 50  0000 L CNN
 F 2 "Capacitor_SMD:C_0805_2012Metric_Pad1.15x1.40mm_HandSolder" H 1638 6750 50  0001 C CNN
@@
 AR Path="/5D249131/5D96E8FA" Ref="C?"  Part="1"
 AR Path="/5D96E8FA" Ref="C?"  Part="1"
-AR Path="/5F050CC1/5D96E8FA" Ref="C?"  Part="1"
-F 0 "C?" H 1315 6946 50  0000 L CNN
+AR Path="/5F050CC1/5D96E8FA" Ref="C74"  Part="1"
+F 0 "C74" H 1315 6946 50  0000 L CNN
 F 1 "1uF" H 1315 6855 50  0000 L CNN
 F 2 "Capacitor_SMD:C_0805_2012Metric_Pad1.15x1.40mm_HandSolder" H 1238 6750 50  0001 C CNN
@@
 AR Path="/5D249131/5D96E95A" Ref="C?"  Part="1"
 AR Path="/5D96E95A" Ref="C?"  Part="1"
-AR Path="/5F050CC1/5D96E95A" Ref="C?"  Part="1"
-F 0 "C?" H 965 6946 50  0000 L CNN
+AR Path="/5F050CC1/5D96E95A" Ref="C73"  Part="1"
+F 0 "C73" H 965 6946 50  0000 L CNN
 F 1 "10uF" H 965 6855 50  0000 L CNN
 F 2 "Capacitor_SMD:C_0805_2012Metric_Pad1.15x1.40mm_HandSolder" H 888 6750 50  0001 C CNN
@@
 AR Path="/5D249131/5D96EB5D" Ref="C?"  Part="1"
 AR Path="/5D96EB5D" Ref="C?"  Part="1"
-AR Path="/5F050CC1/5D96EB5D" Ref="C?"  Part="1"
-F 0 "C?" H 4515 1696 50  0000 L CNN
+AR Path="/5F050CC1/5D96EB5D" Ref="C82"  Part="1"
+F 0 "C82" H 4515 1696 50  0000 L CNN
 F 1 "10uF" H 4515 1605 50  0000 L CNN
 F 2 "Capacitor_SMD:C_0805_2012Metric_Pad1.15x1.40mm_HandSolder" H 4438 1500 50  0001 C CNN
