File: Hardware/AFE Test design PCB/AlternativeDesign2.sch (KiCad schematic (older format))
At the start: 11 parts

Commit message: update
Parts:
- gave numbers to parts that had none: 11
Changed lines of the file:
@@
 AR Path="/5D249182/5D8112F9" Ref="U?"  Part="1"
 AR Path="/5D8112F9" Ref="U?"  Part="1"
-AR Path="/6BC99DBF/5D8112F9" Ref="U?"  Part="1"
-F 0 "U?" H 5100 3575 60  0000 L CNN
+AR Path="/6BC99DBF/5D8112F9" Ref="U6"  Part="1"
+F 0 "U6" H 5100 3575 60  0000 L CNN
 F 1 "INA333AIDGKR" H 5075 2825 60  0000 L CNN
 F 2 "Package_SO:MSOP-8_3x3mm_P0.65mm" H 5200 3600 60  0001 L CNN
@@
 AR Path="/5D249182/5D811300" Ref="C?"  Part="1"
 AR Path="/5D811300" Ref="C?"  Part="1"
-AR Path="/6BC99DBF/5D811300" Ref="C?"  Part="1"
-F 0 "C?" H 4215 4046 50  0000 L CNN
+AR Path="/6BC99DBF/5D811300" Ref="C29"  Part="1"
+F 0 "C29" H 4215 4046 50  0000 L CNN
 F 1 "10uF" H 4215 3955 50  0000 L CNN
 F 2 "Capacitor_SMD:C_0805_2012Metric_Pad1.15x1.40mm_HandSolder" H 4138 3850 50  0001 C CNN
@@
 AR Path="/5D249182/5D811307" Ref="R?"  Part="1"
 AR Path="/5D811307" Ref="R?"  Part="1"
-AR Path="/6BC99DBF/5D811307" Ref="R?"  Part="1"
-F 0 "R?" H 4445 4046 50  0000 L CNN
+AR Path="/6BC99DBF/5D811307" Ref="R42"  Part="1"
+F 0 "R42" H 4445 4046 50  0000 L CNN
 F 1 "1300R" H 4445 3955 50  0000 L CNN
 F 2 "Resistor_SMD:R_0805_2012Metric_Pad1.15x1.40mm_HandSolder" V 4305 4000 50  0001 C CNN
@@
 AR Path="/5D249182/5D811316" Ref="C?"  Part="1"
 AR Path="/5D811316" Ref="C?"  Part="1"
-AR Path="/6BC99DBF/5D811316" Ref="C?"  Part="1"
-F 0 "C?" H 5490 3096 50  0000 L CNN
+AR Path="/6BC99DBF/5D811316" Ref="C30"  Part="1"
+F 0 "C30" H 5490 3096 50  0000 L CNN
 F 1 "100n" H 5490 3005 50  0000 L CNN
 F 2 "Capacitor_SMD:C_0805_2012Metric_Pad1.15x1.40mm_HandSolder" H 5413 2900 50  0001 C CNN
@@
 AR Path="/5D249182/5D81131D" Ref="#PWR?"  Part="1"
 AR Path="/5D81131D" Ref="#PWR?"  Part="1"
-AR Path="/6BC99DBF/5D81131D" Ref="#PWR?"  Part="1"
-F 0 "#PWR?" H 5650 2800 50  0001 C CNN
+AR Path="/6BC99DBF/5D81131D" Ref="#PWR027"  Part="1"
+F 0 "#PWR027" H 5650 2800 50  0001 C CNN
 F 1 "GND" H 5655 2877 50  0000 C CNN
 F 2 "" H 5650 3050 50  0001 C CNN
@@
 AR Path="/5D249182/5D811326" Ref="C?"  Part="1"
 AR Path="/5D811326" Ref="C?"  Part="1"
-AR Path="/6BC99DBF/5D811326" Ref="C?"  Part="1"
-F 0 "C?" H 5490 4221 50  0000 L CNN
+AR Path="/6BC99DBF/5D811326" Ref="C31"  Part="1"
+F 0 "C31" H 5490 4221 50  0000 L CNN
 F 1 "100n" H 5490 4130 50  0000 L CNN
 F 2 "Capacitor_SMD:C_0805_2012Metric_Pad1.15x1.40mm_HandSolder" H 5413 4025 50  0001 C CNN
@@
 AR Path="/5D249182/5D81132D" Ref="#PWR?"  Part="1"
 AR Path="/5D81132D" Ref="#PWR?"  Part="1"
-AR Path="/6BC99DBF/5D81132D" Ref="#PWR?"  Part="1"
-F 0 "#PWR?" H 5650 3925 50  0001 C CNN
+AR Path="/6BC99DBF/5D81132D" Ref="#PWR028"  Part="1"
+F 0 "#PWR028" H 5650 3925 50  0001 C CNN
 F 1 "GND" H 5655 4002 50  0000 C CNN
 F 2 "" H 5650 4175 50  0001 C CNN
@@
 AR Path="/5D249182/5D811337" Ref="#PWR?"  Part="1"
 AR Path="/5D811337" Ref="#PWR?"  Part="1"
-AR Path="/6BC99DBF/5D811337" Ref="#PWR?"  Part="1"
-F 0 "#PWR?" H 4100 3350 50  0001 C CNN
+AR Path="/6BC99DBF/5D811337" Ref="#PWR026"  Part="1"
+F 0 "#PWR026" H 4100 3350 50  0001 C CNN
 F 1 "GND" H 4105 3427 50  0000 C CNN
 F 2 "" H 4100 3600 50  0001 C CNN
@@
 AR Path="/5D249182/5D811340" Ref="R?"  Part="1"
 AR Path="/5D811340" Ref="R?"  Part="1"
-AR Path="/6BC99DBF/5D811340" Ref="R?"  Part="1"
-F 0 "R?" H 3720 3446 50  0000 L CNN
+AR Path="/6BC99DBF/5D811340" Ref="R36"  Part="1"
+F 0 "R36" H 3720 3446 50  0000 L CNN
 F 1 "100k" H 3720 3355 50  0000 L CNN
 F 2 "Resistor_SMD:R_0805_2012Metric_Pad1.15x1.40mm_HandSolder" V 3580 3400 50  0001 C CNN
@@
 AR Path="/5D249182/5D811348" Ref="R?"  Part="1"
 AR Path="/5D811348" Ref="R?"  Part="1"
-AR Path="/6BC99DBF/5D811348" Ref="R?"  Part="1"
-F 0 "R?" H 3720 3546 50  0000 L CNN
+AR Path="/6BC99DBF/5D811348" Ref="R41"  Part="1"
+F 0 "R41" H 3720 3546 50  0000 L CNN
 F 1 "100k" H 3720 3455 50  0000 L CNN
 F 2 "Resistor_SMD:R_0805_2012Metric_Pad1.15x1.40mm_HandSolder" V 3580 3500 50  0001 C CNN
@@
 AR Path="/5D249182/5D811353" Ref="R?"  Part="1"
 AR Path="/5D811353" Ref="R?"  Part="1"
-AR Path="/6BC99DBF/5D811353" Ref="R?"  Part="1"
-F 0 "R?" H 6170 3646 50  0000 L CNN
+AR Path="/6BC99DBF/5D811353" Ref="R47"  Part="1"
+F 0 "R47" H 6170 3646 50  0000 L CNN
 F 1 "1K" H 6170 3555 50  0000 L CNN
 F 2 "Resistor_SMD:R_0805_2012Metric_Pad1.15x1.40mm_HandSolder" V 6030 3600 50  0001 C CNN
@@
 AR Path="/5D249182/5D81135A" Ref="C?"  Part="1"
 AR Path="/5D81135A" Ref="C?"  Part="1"
-AR Path="/6BC99DBF/5D81135A" Ref="C?"  Part="1"
-F 0 "C?" H 6815 3921 50  0000 L CNN
+AR Path="/6BC99DBF/5D81135A" Ref="C32"  Part="1"
+F 0 "C32" H 6815 3921 50  0000 L CNN
 F 1 "100n" H 6815 3830 50  0000 L CNN
 F 2 "Capacitor_SMD:C_0805_2012Metric_Pad1.15x1.40mm_HandSolder" H 6738 3725 50  0001 C CNN
@@
 AR Path="/5D249182/5D811363" Ref="#PWR?"  Part="1"
 AR Path="/5D811363" Ref="#PWR?"  Part="1"
-AR Path="/6BC99DBF/5D811363" Ref="#PWR?"  Part="1"
-F 0 "#PWR?" H 6700 3975 50  0001 C CNN
+AR Path="/6BC99DBF/5D811363" Ref="#PWR029"  Part="1"
+F 0 "#PWR029" H 6700 3975 50  0001 C CNN
 F 1 "GND" H 6705 4052 50  0000 C CNN
 F 2 "" H 6700 4225 50  0001 C CNN
@@
 P 7825 3600
 AR Path="/5D81136E" Ref="JP?"  Part="1"
-AR Path="/6BC99DBF/5D81136E" Ref="JP?"  Part="1"
-F 0 "JP?" H 7825 3864 50  0000 C CNN
+AR Path="/6BC99DBF/5D81136E" Ref="JP23"  Part="1"
+F 0 "JP23" H 7825 3864 50  0000 C CNN
 F 1 "Jumper" H 7825 3773 50  0000 C CNN
 F 2 "Jumper:SolderJumper-2_P1.3mm_Open_Pad1.0x1.5mm" H 7825 3600 50  0001 C CNN
@@
 P 7400 3500
 AR Path="/5D811377" Ref="TP?"  Part="1"
-AR Path="/6BC99DBF/5D811377" Ref="TP?"  Part="1"
-F 0 "TP?" H 7400 3825 50  0000 L CNN
+AR Path="/6BC99DBF/5D811377" Ref="TP15"  Part="1"
+F 0 "TP15" H 7400 3825 50  0000 L CNN
 F 1 "TestPoint" H 7400 3725 50  0000 L CNN
 F 2 "TestPoint:TestPoint_THTPad_1.5x1.5mm_Drill0.7mm" H 7600 3500 50  0001 C CNN
