File: Hardware/AFE Test design PCB/EMG12.sch (KiCad schematic (older format))
At the start: 25 parts

Commit message: update
Parts:
- R10: renamed from R?; value 30k -> 27k
- R4: renamed from R?; value 160k -> 180k
- R6: renamed from R?; value 620k -> 510k
- R9: renamed from R?; value 10k -> 18k
- gave numbers to parts that had none: 21
Changed lines of the file:
@@
 AR Path="/6DE5C03E/6DE65F14" Ref="C?"  Part="1"
 AR Path="/6DF2C954/6DE65F14" Ref="C?"  Part="1"
-AR Path="/794AF32B/6DE65F14" Ref="C?"  Part="1"
-F 0 "C?" V 6400 2225 50  0000 C CNN
+AR Path="/794AF32B/6DE65F14" Ref="C6"  Part="1"
+F 0 "C6" V 6400 2225 50  0000 C CNN
 F 1 "4700nF" V 6700 2225 50  0000 C CNN
 F 2 "Capacitor_SMD:C_0805_2012Metric_Pad1.15x1.40mm_HandSolder" H 6588 2075 50  0001 C CNN
@@
 AR Path="/6DE5C03E/6DE65F80" Ref="C?"  Part="1"
 AR Path="/6DF2C954/6DE65F80" Ref="C?"  Part="1"
-AR Path="/794AF32B/6DE65F80" Ref="C?"  Part="1"
-F 0 "C?" H 5335 3579 50  0000 R CNN
+AR Path="/794AF32B/6DE65F80" Ref="C2"  Part="1"
+F 0 "C2" H 5335 3579 50  0000 R CNN
 F 1 "1nF" H 5335 3670 50  0000 R CNN
 F 2 "Capacitor_SMD:C_0805_2012Metric_Pad1.15x1.40mm_HandSolder" H 5488 3475 50  0001 C CNN
@@
 AR Path="/6DE5C03E/6DE65F8E" Ref="M?"  Part="1"
 AR Path="/6DF2C954/6DE65F8E" Ref="M?"  Part="1"
-AR Path="/794AF32B/6DE65F8E" Ref="M?"  Part="1"
-F 0 "M?" H 6575 6385 45  0000 C CNN
+AR Path="/794AF32B/6DE65F8E" Ref="M1"  Part="1"
+F 0 "M1" H 6575 6385 45  0000 C CNN
 F 1 "AD8232" H 6575 6301 45  0000 C CNN
 F 2 "Package_CSP:LFCSP-20-1EP_4x4mm_P0.5mm_EP2.1x2.1mm" H 6575 6225 20  0001 C CNN
@@
 AR Path="/6DE5C03E/6DE65FBC" Ref="C?"  Part="1"
 AR Path="/6DF2C954/6DE65FBC" Ref="C?"  Part="1"
-AR Path="/794AF32B/6DE65FBC" Ref="C?"  Part="1"
-F 0 "C?" H 7360 4029 50  0000 R CNN
+AR Path="/794AF32B/6DE65FBC" Ref="C7"  Part="1"
+F 0 "C7" H 7360 4029 50  0000 R CNN
 F 1 "100nF" H 7360 4120 50  0000 R CNN
 F 2 "Capacitor_SMD:C_0805_2012Metric_Pad1.15x1.40mm_HandSolder" H 7513 3925 50  0001 C CNN
@@
 AR Path="/6DE5C03E/78732C38" Ref="R?"  Part="1"
 AR Path="/6DF2C954/78732C38" Ref="R?"  Part="1"
-AR Path="/794AF32B/78732C38" Ref="R?"  Part="1"
-F 0 "R?" V 5350 3025 50  0000 C CNN
+AR Path="/794AF32B/78732C38" Ref="R7"  Part="1"
+F 0 "R7" V 5350 3025 50  0000 C CNN
 F 1 "180k" V 5250 3025 50  0000 C CNN
 F 2 "Resistor_SMD:R_0805_2012Metric_Pad1.15x1.40mm_HandSolder" V 5280 3025 50  0001 C CNN
@@
 AR Path="/6DE5C03E/78732C39" Ref="R?"  Part="1"
 AR Path="/6DF2C954/78732C39" Ref="R?"  Part="1"
-AR Path="/794AF32B/78732C39" Ref="R?"  Part="1"
-F 0 "R?" V 5350 3225 50  0000 C CNN
+AR Path="/794AF32B/78732C39" Ref="R8"  Part="1"
+F 0 "R8" V 5350 3225 50  0000 C CNN
 F 1 "180k" V 5450 3225 50  0000 C CNN
 F 2 "Resistor_SMD:R_0805_2012Metric_Pad1.15x1.40mm_HandSolder" V 5280 3225 50  0001 C CNN
@@
 AR Path="/6DE5C03E/6DE65FD2" Ref="R?"  Part="1"
 AR Path="/6DF2C954/6DE65FD2" Ref="R?"  Part="1"
-AR Path="/794AF32B/6DE65FD2" Ref="R?"  Part="1"
-F 0 "R?" V 4943 3825 50  0000 C CNN
+AR Path="/794AF32B/6DE65FD2" Ref="R5"  Part="1"
+F 0 "R5" V 4943 3825 50  0000 C CNN
 F 1 "390k" V 5034 3825 50  0000 C CNN
 F 2 "Resistor_SMD:R_0805_2012Metric_Pad1.15x1.40mm_HandSolder" V 5080 3825 50  0001 C CNN
@@
 AR Path="/6DE5C03E/6DE65FF3" Ref="R?"  Part="1"
 AR Path="/6DF2C954/6DE65FF3" Ref="R?"  Part="1"
-AR Path="/794AF32B/6DE65FF3" Ref="R?"  Part="1"
-F 0 "R?" V 7825 3450 50  0000 L CNN
+AR Path="/794AF32B/6DE65FF3" Ref="R12"  Part="1"
+F 0 "R12" V 7825 3450 50  0000 L CNN
 F 1 "10M" V 7700 3450 50  0000 L CNN
 F 2 "Resistor_SMD:R_0805_2012Metric_Pad1.15x1.40mm_HandSolder" V 7755 3525 50  0001 C CNN
@@
 AR Path="/6DE5C03E/6DE65FFA" Ref="R?"  Part="1"
 AR Path="/6DF2C954/6DE65FFA" Ref="R?"  Part="1"
-AR Path="/794AF32B/6DE65FFA" Ref="R?"  Part="1"
-F 0 "R?" V 7475 3650 50  0000 L CNN
+AR Path="/794AF32B/6DE65FFA" Ref="R11"  Part="1"
+F 0 "R11" V 7475 3650 50  0000 L CNN
 F 1 "10M" V 7575 3650 50  0000 L CNN
 F 2 "Resistor_SMD:R_0805_2012Metric_Pad1.15x1.40mm_HandSolder" V 7405 3725 50  0001 C CNN
@@
 AR Path="/6DE5C03E/78732C3D" Ref="C?"  Part="1"
 AR Path="/6DF2C954/78732C3D" Ref="C?"  Part="1"
-AR Path="/794AF32B/78732C3D" Ref="C?"  Part="1"
-F 0 "C?" V 7800 3550 50  0000 C CNN
+AR Path="/794AF32B/78732C3D" Ref="C8"  Part="1"
+F 0 "C8" V 7800 3550 50  0000 C CNN
 F 1 "100nF" V 7900 3525 50  0000 C CNN
 F 2 "Capacitor_SMD:C_0805_2012Metric_Pad1.15x1.40mm_HandSolder" H 7888 3575 50  0001 C CNN
@@
 AR Path="/6DE5C03E/78732C3F" Ref="TP?"  Part="1"
 AR Path="/6DF2C954/78732C3F" Ref="TP?"  Part="1"
-AR Path="/794AF32B/78732C3F" Ref="TP?"  Part="1"
-F 0 "TP?" H 4725 4000 50  0000 C CNN
+AR Path="/794AF32B/78732C3F" Ref="TP3"  Part="1"
+F 0 "TP3" H 4725 4000 50  0000 C CNN
 F 1 "TestPoint" H 4725 3900 50  0000 C CNN
 F 2 "TestPoint:TestPoint_THTPad_1.5x1.5mm_Drill0.7mm" H 4925 3675 50  0001 C CNN
@@
 P 4725 2750
 AR Path="/6DE5C03E/78732C40" Ref="JP?"  Part="1"
-AR Path="/794AF32B/78732C40" Ref="JP?"  Part="1"
-F 0 "JP?" V 4771 2662 50  0000 R CNN
+AR Path="/794AF32B/78732C40" Ref="JP10"  Part="1"
+F 0 "JP10" V 4771 2662 50  0000 R CNN
 F 1 "Jumper_2_Open" V 4680 2662 50  0000 R CNN
 F 2 "Jumper:SolderJumper-2_P1.3mm_Open_Pad1.0x1.5mm" H 4725 2750 50  0001 C CNN
@@
 AR Path="/6DE5C03E/78732C41" Ref="TP?"  Part="1"
 AR Path="/6DF2C954/78732C41" Ref="TP?"  Part="1"
-AR Path="/794AF32B/78732C41" Ref="TP?"  Part="1"
-F 0 "TP?" H 4725 2225 50  0000 C CNN
+AR Path="/794AF32B/78732C41" Ref="TP2"  Part="1"
+F 0 "TP2" H 4725 2225 50  0000 C CNN
 F 1 "TestPoint" H 4725 2125 50  0000 C CNN
 F 2 "TestPoint:TestPoint_THTPad_1.5x1.5mm_Drill0.7mm" H 4925 1875 50  0001 C CNN
@@
 AR Path="/6DE5C03E/78732C43" Ref="R?"  Part="1"
 AR Path="/6DF2C954/78732C43" Ref="R?"  Part="1"
-AR Path="/794AF32B/78732C43" Ref="R?"  Part="1"
-F 0 "R?" H 8245 3021 50  0000 L CNN
+AR Path="/794AF32B/78732C43" Ref="R14"  Part="1"
+F 0 "R14" H 8245 3021 50  0000 L CNN
 F 1 "340k" H 8245 2930 50  0000 L CNN
 F 2 "Resistor_SMD:R_0805_2012Metric_Pad1.15x1.40mm_HandSolder" V 8105 2975 50  0001 C CNN
@@
 AR Path="/6DE5C03E/78732C3E" Ref="TP?"  Part="1"
 AR Path="/6DF2C954/78732C3E" Ref="TP?"  Part="1"
-AR Path="/794AF32B/78732C3E" Ref="TP?"  Part="1"
+AR Path="/794AF32B/78732C3E" Ref="TP1"  Part="1"
 AR Path="/78732C3E" Ref="TP?"  Part="1"
-F 0 "TP?" H 4583 5545 50  0000 L CNN
+F 0 "TP1" H 4583 5545 50  0000 L CNN
 F 1 "TestPoint" H 4583 5454 50  0000 L CNN
 F 2 "TestPoint:TestPoint_THTPad_1.5x1.5mm_Drill0.7mm" H 4725 5425 50  0001 C CNN
@@
 	5450 5025 5450 5075
 $Comp
-L Device:R R?
+L Device:R R10
 U 1 1 785A8500
 P 5450 5225
-F 0 "R?" H 5520 5271 50  0000 L CNN
-F 1 "30k" H 5520 5180 50  0000 L CNN
+F 0 "R10" H 5520 5271 50  0000 L CNN
+F 1 "27k" H 5520 5180 50  0000 L CNN
 F 2 "Resistor_SMD:R_0805_2012Metric_Pad1.15x1.40mm_HandSolder" V 5380 5225 50  0001 C CNN
 F 3 "~" H 5450 5225 50  0001 C CNN
@@
 	5450 5375 5450 5425
 $Comp
-L Device:R R?
+L Device:R R6
 U 1 1 785A878B
 P 5150 4225
-F 0 "R?" V 4943 4225 50  0000 C CNN
-F 1 "620k" V 5034 4225 50  0000 C CNN
+F 0 "R6" V 4943 4225 50  0000 C CNN
+F 1 "510k" V 5034 4225 50  0000 C CNN
 F 2 "Resistor_SMD:R_0805_2012Metric_Pad1.15x1.40mm_HandSolder" V 5080 4225 50  0001 C CNN
 F 3 "~" H 5150 4225 50  0001 C CNN
@@
 AR Path="/6DE5C03E/785A882E" Ref="C?"  Part="1"
 AR Path="/6DF2C954/785A882E" Ref="C?"  Part="1"
-AR Path="/794AF32B/785A882E" Ref="C?"  Part="1"
-F 0 "C?" H 5335 4379 50  0000 R CNN
+AR Path="/794AF32B/785A882E" Ref="C3"  Part="1"
+F 0 "C3" H 5335 4379 50  0000 R CNN
 F 1 "1nF" H 5335 4470 50  0000 R CNN
 F 2 "Capacitor_SMD:C_0805_2012Metric_Pad1.15x1.40mm_HandSolder" H 5488 4275 50  0001 C CNN
@@
 AR Path="/6DE5C03E/785A887C" Ref="C?"  Part="1"
 AR Path="/6DF2C954/785A887C" Ref="C?"  Part="1"
-AR Path="/794AF32B/785A887C" Ref="C?"  Part="1"
-F 0 "C?" H 4610 4554 50  0000 R CNN
+AR Path="/794AF32B/785A887C" Ref="C1"  Part="1"
+F 0 "C1" H 4610 4554 50  0000 R CNN
 F 1 "1nF" H 4610 4645 50  0000 R CNN
 F 2 "Capacitor_SMD:C_0805_2012Metric_Pad1.15x1.40mm_HandSolder" H 4763 4450 50  0001 C CNN
@@
 $EndComp
 $Comp
-L Device:R R?
+L Device:R R4
 U 1 1 785A88D0
 P 4725 3975
-F 0 "R?" H 4655 3929 50  0000 R CNN
-F 1 "160k" H 4655 4020 50  0000 R CNN
+F 0 "R4" H 4655 3929 50  0000 R CNN
+F 1 "180k" H 4655 4020 50  0000 R CNN
 F 2 "Resistor_SMD:R_0805_2012Metric_Pad1.15x1.40mm_HandSolder" V 4655 3975 50  0001 C CNN
 F 3 "~" H 4725 3975 50  0001 C CNN
@@
 	5450 4625 5775 4625
 $Comp
-L Device:R R?
+L Device:R R9
 U 1 1 785B17E7
 P 5450 4825
-F 0 "R?" H 5520 4871 50  0000 L CNN
-F 1 "10k" H 5520 4780 50  0000 L CNN
+F 0 "R9" H 5520 4871 50  0000 L CNN
+F 1 "18k" H 5520 4780 50  0000 L CNN
 F 2 "Resistor_SMD:R_0805_2012Metric_Pad1.15x1.40mm_HandSolder" V 5380 4825 50  0001 C CNN
 F 3 "~" H 5450 4825 50  0001 C CNN
@@
 AR Path="/6DE5C03E/7874AAA5" Ref="C?"  Part="1"
 AR Path="/6DF2C954/7874AAA5" Ref="C?"  Part="1"
-AR Path="/794AF32B/7874AAA5" Ref="C?"  Part="1"
-F 0 "C?" V 8350 3225 50  0000 C CNN
+AR Path="/794AF32B/7874AAA5" Ref="C9"  Part="1"
+F 0 "C9" V 8350 3225 50  0000 C CNN
 F 1 "4700nF" V 8650 3225 50  0000 C CNN
 F 2 "Capacitor_SMD:C_0805_2012Metric_Pad1.15x1.40mm_HandSolder" H 8538 3075 50  0001 C CNN
@@
 AR Path="/6DE5C03E/7874CFB6" Ref="R?"  Part="1"
 AR Path="/6DF2C954/7874CFB6" Ref="R?"  Part="1"
-AR Path="/794AF32B/7874CFB6" Ref="R?"  Part="1"
-F 0 "R?" H 9245 2846 50  0000 L CNN
+AR Path="/794AF32B/7874CFB6" Ref="R15"  Part="1"
+F 0 "R15" H 9245 2846 50  0000 L CNN
 F 1 "3.4k" H 9245 2755 50  0000 L CNN
 F 2 "Resistor_SMD:R_0805_2012Metric_Pad1.15x1.40mm_HandSolder" V 9105 2800 50  0001 C CNN
@@
 AR Path="/6DE5C03E/5F1825CC" Ref="TP?"  Part="1"
 AR Path="/6DF2C954/5F1825CC" Ref="TP?"  Part="1"
-AR Path="/794AF32B/5F1825CC" Ref="TP?"  Part="1"
-F 0 "TP?" V 7670 3174 50  0000 C CNN
+AR Path="/794AF32B/5F1825CC" Ref="TP4"  Part="1"
+F 0 "TP4" V 7670 3174 50  0000 C CNN
 F 1 "TestPoint" V 7579 3174 50  0000 C CNN
 F 2 "TestPoint:TestPoint_THTPad_1.5x1.5mm_Drill0.7mm" H 7675 3100 50  0001 C CNN
@@
 P 7825 3225
 AR Path="/6DE5C03E/68F56670" Ref="JP?"  Part="1"
-AR Path="/794AF32B/68F56670" Ref="JP?"  Part="1"
-F 0 "JP?" H 7850 3825 50  0000 R CNN
+AR Path="/794AF32B/68F56670" Ref="JP13"  Part="1"
+F 0 "JP13" H 7850 3825 50  0000 R CNN
 F 1 "Jumper_2_Open" H 8075 3725 50  0000 R CNN
 F 2 "Jumper:SolderJumper-2_P1.3mm_Open_Pad1.0x1.5mm" H 7825 3225 50  0001 C CNN
