File: Hardware/HD-SEMG prototype V2/ADS1298_setup.sch (KiCad schematic (older format))
At the start: 27 parts, among them IC1 ADS1298_By_Oliver, J21 Conn_01x03, J22 Conn_01x03, J24 Conn_01x03, J25 Conn_01x03, U36 357LB3CI002M0480

Commit message: update
Connections:
- net VREFP1: no longer names the net of C35.1, C36.1, IC1.25 (VREFN)
Changed lines of the file:
@@
 Wire Wire Line
 	4075 1600 4500 1600
-Text GLabel 4500 850  1    50   Input ~ 0
-VREFP1
 $Comp
 L Device:C C?
@@
 Wire Wire Line
 	4475 6400 4475 6275
-Wire Wire Line
-	4500 850  4500 1000
-Connection ~ 4500 1000
 Wire Wire Line
 	4500 1000 4500 1150
@@
 	2800 7100 2800 7275
 Connection ~ 4075 1600
-Text GLabel 4500 1725 3    50   Input ~ 0
-VREFN
 Connection ~ 4500 1600
 $Comp
@@
 	4075 1000 4500 1000
 Wire Wire Line
-	4500 1725 4500 1600
-Wire Wire Line
 	4900 2625 4825 2625
