File: Hardware/HD-SEMG prototype V2/_autosave-HDSEMG.kicad_pcb (KiCad board)
At the start: 2 copper layers, 150 x 86.9 mm, 210 parts, among them IC1 ADS1298_By_Oliver, J1 AUDIO_JACK_By_OLIVER, J10 Conn_01x02, J11 Barrel_Jack_Switch, J12 Conn_01x01, J13 Conn_01x03, J14 Conn_01x03, J15 Conn_01x03, J16 Conn_01x03, J17 Conn_01x03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

Commit message: update
Parts:
- removed REF**: KiCad-Logo2_8mm_SilkScreen, Symbol:KiCad-Logo2_8mm_SilkScreen
Connections:
- net VREFP1 renamed Net-(C35-Pad1)
Routing:
- net -2V5: track 113.2 -> 117.3 mm
